File: electronics/sunpowered.sch (KiCad schematic (older format))
At the start: 16 parts

Commit message: corrected current sensor direction
Connections:
- wire segments 45 -> 46
Other:
- moved on the sheet: C?, F?
Changed lines of the file:
@@
 L FUSE F?
 U 1 1 54D5362E
-P 2500 850
-F 0 "F?" H 2600 900 50  0000 C CNN
-F 1 "8A" H 2400 800 50  0000 C CNN
-F 2 "" H 2500 850 60  0000 C CNN
-F 3 "" H 2500 850 60  0000 C CNN
-	1    2500 850
+P 2550 850
+F 0 "F?" H 2650 900 50  0000 C CNN
+F 1 "8A" H 2450 800 50  0000 C CNN
+F 2 "" H 2550 850 60  0000 C CNN
+F 3 "" H 2550 850 60  0000 C CNN
+	1    2550 850
 	1    0    0    -1
 $EndComp
@@
 L +5P #PWR03
 U 1 1 54D71F91
-P 3800 1250
-F 0 "#PWR03" H 3800 1100 60  0001 C CNN
-F 1 "+5P" H 3800 1390 60  0000 C CNN
-F 2 "" H 3800 1250 60  0000 C CNN
-F 3 "" H 3800 1250 60  0000 C CNN
-	1    3800 1250
+P 2550 1300
+F 0 "#PWR03" H 2550 1150 60  0001 C CNN
+F 1 "+5P" H 2550 1440 60  0000 C CNN
+F 2 "" H 2550 1300 60  0000 C CNN
+F 3 "" H 2550 1300 60  0000 C CNN
+	1    2550 1300
 	1    0    0    -1
 $EndComp
@@
 P 3200 1500
 F 0 "IC?" V 3400 1850 50  0000 L CNN
-F 1 "ACS713" V 3600 1750 50  0000 L CNN
+F 1 "ACS713" V 3050 850 50  0000 L CNN
 F 2 "Housings_SOIC:SOIC-8_3.9x4.9mm_Pitch1.27mm" H 3200 1500 50  0001 C CIN
 F 3 "http://www.allegromicro.com/en/Products/Part_Numbers/0713/0713.pdf" H 3300 1950 60  0001 C CNN
 F 4 "Current sensor" V 2950 950 39  0000 C CNN "Note"
 	1    3200 1500
-	0    1    1    0
+	0    -1   1    0
 $EndComp
 $Comp
 L C C?
 U 1 1 54D74223
-P 3800 1800
-F 0 "C?" H 3850 1900 50  0000 L CNN
-F 1 "0.1uF" H 3850 1700 50  0000 L CNN
-F 2 "" H 3838 1650 30  0000 C CNN
-F 3 "" H 3800 1800 60  0000 C CNN
-	1    3800 1800
+P 2550 1700
+F 0 "C?" H 2400 1800 50  0000 L CNN
+F 1 "0.1uF" H 2300 1550 50  0000 L CNN
+F 2 "" H 2588 1550 30  0000 C CNN
+F 3 "" H 2550 1700 60  0000 C CNN
+	1    2550 1700
 	1    0    0    -1
 $EndComp
@@
 	6350 850  7800 850
 Wire Wire Line
-	2050 2000 2700 2000
-Wire Wire Line
-	2700 2000 4250 2000
-Wire Wire Line
-	4250 2000 4650 2000
-Wire Wire Line
-	4650 2000 5050 2000
-Wire Wire Line
-	5050 2000 5400 2000
-Wire Wire Line
-	5400 2000 5800 2000
-Wire Wire Line
-	5800 2000 7800 2000
-Wire Wire Line
 	7550 2000 7550 1700
 Connection ~ 4250 850
@@
 Connection ~ 3400 850
 Wire Wire Line
-	3100 1900 3100 2350
-Wire Wire Line
-	3400 1900 3400 2350
+	3000 1900 3000 2350
+Wire Wire Line
+	3300 1900 3300 2350
 Wire Wire Line
 	6750 1500 6400 1500
 Wire Wire Line
-	6400 1500 6400 2300
+	6400 1500 6400 2350
 Wire Wire Line
 	3300 850  3400 850
@@
 	5800 850  6200 850
 Wire Wire Line
-	2750 850  3000 850
+	2800 850  3000 850
 Wire Wire Line
 	3000 850  3100 850
 Wire Wire Line
-	3600 1500 3800 1500
-Wire Wire Line
-	2050 850  2250 850
-Wire Wire Line
-	3800 1250 3800 1500
-Wire Wire Line
-	3800 1500 3800 1600
+	2050 850  2300 850
 Wire Wire Line
 	2050 1750 2050 2000
@@
 Wire Wire Line
 	3400 850  3400 1100
-Connection ~ 3800 1500
-Wire Wire Line
-	2800 1500 2700 1500
-Wire Wire Line
-	2700 1500 2700 2000
-Connection ~ 2700 2000
+Wire Wire Line
+	2550 1500 2800 1500
 Wire Wire Line
 	4250 950  4250 850
@@
 Connection ~ 6750 2000
 Connection ~ 6750 1500
+Wire Wire Line
+	2550 1300 2550 1500
+Wire Wire Line
+	2550 1900 2550 2000
+Connection ~ 2550 2000
+Wire Wire Line
+	3600 1500 3750 1500
+Wire Wire Line
+	3750 1500 3750 1650
+$Comp
+L GND #PWR?
+U 1 1 54D76516
+P 3750 1650
+F 0 "#PWR?" H 3750 1400 60  0001 C CNN
+F 1 "GND" H 3750 1500 60  0000 C CNN
+F 2 "" H 3750 1650 60  0000 C CNN
+F 3 "" H 3750 1650 60  0000 C CNN
+	1    3750 1650
+	1    0    0    -1
+$EndComp
+Wire Wire Line
+	2050 2000 2550 2000
+Wire Wire Line
+	2550 2000 4250 2000
+Wire Wire Line
+	4250 2000 4650 2000
+Wire Wire Line
+	4650 2000 5050 2000
+Wire Wire Line
+	5050 2000 5400 2000
+Wire Wire Line
+	5400 2000 5800 2000
+Wire Wire Line
+	5800 2000 6750 2000
+Wire Wire Line
+	6750 2000 7550 2000
 $EndSCHEMATC

Commit message: global in/out labels added for the input stage
Parts:
- added C?: 47n, symbol C
- C?: value 0.1uF -> 0.1u
Connections:
- net labels added: PanelCurrentSense, PowerOn
- wire segments 46 -> 34
Changed lines of the file:
@@
 P 2550 1700
 F 0 "C?" H 2400 1800 50  0000 L CNN
-F 1 "0.1uF" H 2300 1550 50  0000 L CNN
+F 1 "0.1u" H 2300 1550 50  0000 L CNN
 F 2 "" H 2588 1550 30  0000 C CNN
 F 3 "" H 2550 1700 60  0000 C CNN
@@
 Connection ~ 5050 2000
 Wire Wire Line
-	5050 1500 5400 1500
-Wire Wire Line
-	5400 1500 5650 1500
+	5050 1500 5650 1500
 Wire Wire Line
 	5400 2000 5400 1900
@@
 	3000 1900 3000 2350
 Wire Wire Line
-	3300 1900 3300 2350
-Wire Wire Line
 	6750 1500 6400 1500
 Wire Wire Line
 	6400 1500 6400 2350
 Wire Wire Line
-	3300 850  3400 850
+	3300 850  6200 850
 Wire Wire Line
-	3400 850  4250 850
-Wire Wire Line
-	4250 850  4650 850
-Wire Wire Line
-	4650 850  5050 850
-Wire Wire Line
-	5050 850  5800 850
-Wire Wire Line
-	5800 850  6200 850
-Wire Wire Line
-	2800 850  3000 850
-Wire Wire Line
-	3000 850  3100 850
+	2800 850  3100 850
 Wire Wire Line
 	2050 850  2300 850
@@
 	3600 1500 3750 1500
 Wire Wire Line
-	3750 1500 3750 1650
+	3750 1500 3750 2600
 $Comp
 L GND #PWR?
 U 1 1 54D76516
-P 3750 1650
-F 0 "#PWR?" H 3750 1400 60  0001 C CNN
-F 1 "GND" H 3750 1500 60  0000 C CNN
-F 2 "" H 3750 1650 60  0000 C CNN
-F 3 "" H 3750 1650 60  0000 C CNN
-	1    3750 1650
+P 3750 2600
+F 0 "#PWR?" H 3750 2350 60  0001 C CNN
+F 1 "GND" H 3750 2450 60  0000 C CNN
+F 2 "" H 3750 2600 60  0000 C CNN
+F 3 "" H 3750 2600 60  0000 C CNN
+	1    3750 2600
 	1    0    0    -1
 $EndComp
 Wire Wire Line
-	2050 2000 2550 2000
+	2050 2000 7550 2000
 Wire Wire Line
-	2550 2000 4250 2000
+	3300 1900 3300 2200
+$Comp
+L C C?
+U 1 1 54D76924
+P 3300 2400
+F 0 "C?" H 3350 2500 50  0000 L CNN
+F 1 "47n" H 3350 2300 50  0000 L CNN
+F 2 "" H 3338 2250 30  0000 C CNN
+F 3 "" H 3300 2400 60  0000 C CNN
+	1    3300 2400
+	1    0    0    -1
+$EndComp
+$Comp
+L GND #PWR?
+U 1 1 54D76957
+P 3300 2600
+F 0 "#PWR?" H 3300 2350 60  0001 C CNN
+F 1 "GND" H 3300 2450 60  0000 C CNN
+F 2 "" H 3300 2600 60  0000 C CNN
+F 3 "" H 3300 2600 60  0000 C CNN
+	1    3300 2600
+	1    0    0    -1
+$EndComp
+Text GLabel 2950 2350 0    60   Output ~ 0
+PanelCurrentSense
 Wire Wire Line
-	4250 2000 4650 2000
+	3000 2350 2950 2350
+Text GLabel 6300 2350 0    60   Input ~ 0
+PowerOn
 Wire Wire Line
-	4650 2000 5050 2000
-Wire Wire Line
-	5050 2000 5400 2000
-Wire Wire Line
-	5400 2000 5800 2000
-Wire Wire Line
-	5800 2000 6750 2000
-Wire Wire Line
-	6750 2000 7550 2000
+	6400 2350 6300 2350
 $EndSCHEMATC

Commit message: current and voltage sense nodes added
Connections:
- net labels added: PanelVoltageSense
- wire segments 34 -> 51
Other:
- moved on the sheet: C?, D?, F?, IC?, Q?, R?, SW?, T?

Commit message: more clear voltage sense lines
Connections:
- net labels added: PanelVoltageSense+, PanelVoltageSense-
- net labels removed: PanelVoltageSense
- wire segments 51 -> 37
Changed lines of the file:
@@
 Connection ~ 5150 2100
 Wire Wire Line
-	5150 1600 5500 1600
-Wire Wire Line
-	5500 1600 5750 1600
+	5150 1600 5750 1600
 Wire Wire Line
 	5500 2100 5500 2000
@@
 	6500 1600 6500 2450
 Wire Wire Line
-	3550 950  3650 950
+	3550 950  6550 950
 Wire Wire Line
-	3650 950  4500 950
-Wire Wire Line
-	4500 950  4750 950
-Wire Wire Line
-	4750 950  5150 950
-Wire Wire Line
-	5150 950  5900 950
-Wire Wire Line
-	5900 950  6550 950
-Wire Wire Line
-	2800 950  3250 950
-Wire Wire Line
-	3250 950  3350 950
+	2800 950  3350 950
 Wire Wire Line
 	2050 950  2300 950
@@
 	2050 1850 2050 2100
 Wire Wire Line
-	3250 700  3250 950
-Wire Wire Line
-	3250 950  3250 1200
+	3250 700  3250 1200
 Connection ~ 3250 950
 Wire Wire Line
@@
 	4000 1600 4000 2700
 Wire Wire Line
-	2050 2100 2550 2100
-Wire Wire Line
-	2550 2100 4500 2100
-Wire Wire Line
-	4500 2100 4750 2100
-Wire Wire Line
-	4750 2100 5150 2100
-Wire Wire Line
-	5150 2100 5500 2100
-Wire Wire Line
-	5500 2100 5900 2100
-Wire Wire Line
-	5900 2100 6850 2100
-Wire Wire Line
-	6850 2100 7650 2100
-Wire Wire Line
-	7650 2100 7900 2100
+	2050 2100 7900 2100
 Wire Wire Line
 	3550 2000 3550 2300
@@
 	6500 2450 6400 2450
 Text GLabel 2950 700  0    60   Output ~ 0
-PanelVoltageSense
+PanelVoltageSense+
 Wire Wire Line
 	2950 700  3250 700
+Text GLabel 2950 2300 0    60   Output ~ 0
+PanelVoltageSense-
+Wire Wire Line
+	2950 2300 3150 2300
+Wire Wire Line
+	3150 2300 3150 2100
+Connection ~ 3150 2100
 $EndSCHEMATC

Commit message: current limit for current sensor chip
Parts:
- added R?: 220, symbol R
Connections:
- wire segments 37 -> 56
Other:
- moved on the sheet: C?, D?, F?, IC?, Q?, R?, SW?, T?

Commit message: minor cleanup
Connections:
- wire segments 56 -> 55
Other:
- moved on the sheet: C?, IC?, R?
Changed lines of the file:
@@
 L +5P #PWR03
 U 1 1 54D71F91
-P 2550 1750
-F 0 "#PWR03" H 2550 1600 60  0001 C CNN
-F 1 "+5P" H 2550 1890 60  0000 C CNN
-F 2 "" H 2550 1750 60  0000 C CNN
-F 3 "" H 2550 1750 60  0000 C CNN
-	1    2550 1750
+P 2500 1700
+F 0 "#PWR03" H 2500 1550 60  0001 C CNN
+F 1 "+5P" H 2500 1840 60  0000 C CNN
+F 2 "" H 2500 1700 60  0000 C CNN
+F 3 "" H 2500 1700 60  0000 C CNN
+	1    2500 1700
 	1    0    0    -1
 $EndComp
@@
 L ACS713ELCTR-30A-T IC?
 U 1 1 54D71B52
-P 3450 1850
-F 0 "IC?" V 3650 2200 50  0000 L CNN
-F 1 "ACS713" V 3300 1200 50  0000 L CNN
-F 2 "Housings_SOIC:SOIC-8_3.9x4.9mm_Pitch1.27mm" H 3450 1850 50  0001 C CIN
-F 3 "http://www.allegromicro.com/en/Products/Part_Numbers/0713/0713.pdf" H 3550 2300 60  0001 C CNN
-F 4 "Current sensor" V 3200 1300 39  0000 C CNN "Note"
-	1    3450 1850
+P 3400 1850
+F 0 "IC?" V 3650 1400 50  0000 L CNN
+F 1 "ACS713" V 3250 1200 50  0000 L CNN
+F 2 "Housings_SOIC:SOIC-8_3.9x4.9mm_Pitch1.27mm" H 3400 1850 50  0001 C CIN
+F 3 "http://www.allegromicro.com/en/Products/Part_Numbers/0713/0713.pdf" H 3500 2300 60  0001 C CNN
+F 4 "Current sensor" V 3150 1300 39  0000 C CNN "Note"
+	1    3400 1850
 	0    -1   1    0
 $EndComp
@@
 L C C?
 U 1 1 54D74223
-P 2550 2300
-F 0 "C?" H 2400 2400 50  0000 L CNN
-F 1 "0.1u" H 2300 2150 50  0000 L CNN
-F 2 "" H 2588 2150 30  0000 C CNN
-F 3 "" H 2550 2300 60  0000 C CNN
-	1    2550 2300
+P 3000 2450
+F 0 "C?" H 2850 2550 50  0000 L CNN
+F 1 "0.1u" H 2800 2350 50  0000 L CNN
+F 2 "" H 3038 2300 30  0000 C CNN
+F 3 "" H 3000 2450 60  0000 C CNN
+	1    3000 2450
 	1    0    0    -1
 $EndComp
@@
 L C C?
 U 1 1 54D76924
-P 3550 2450
-F 0 "C?" H 3600 2550 50  0000 L CNN
-F 1 "47n" H 3600 2350 50  0000 L CNN
-F 2 "" H 3588 2300 30  0000 C CNN
-F 3 "" H 3550 2450 60  0000 C CNN
-	1    3550 2450
-	1    0    0    -1
-$EndComp
-Text GLabel 2950 2950 0    60   Output ~ 0
+P 3500 2450
+F 0 "C?" H 3550 2550 50  0000 L CNN
+F 1 "47n" H 3550 2350 50  0000 L CNN
+F 2 "" H 3538 2300 30  0000 C CNN
+F 3 "" H 3500 2450 60  0000 C CNN
+	1    3500 2450
+	1    0    0    -1
+$EndComp
+Text GLabel 2850 2950 0    60   Output ~ 0
 PanelCurrentSense
 Text GLabel 6400 2950 0    60   Input ~ 0
@@
 Connection ~ 5150 2650
 Wire Wire Line
-	2050 2650 2550 2650
-Wire Wire Line
-	2550 2650 3150 2650
-Wire Wire Line
-	3150 2650 4000 2650
+	2050 2650 3000 2650
+Wire Wire Line
+	3000 2650 3050 2650
+Wire Wire Line
+	3000 2650 3500 2650
+Wire Wire Line
+	3500 2650 4000 2650
 Wire Wire Line
 	4000 2650 4500 2650
@@
 Wire Wire Line
 	6850 2650 7650 2650
-Wire Wire Line
-	7650 2650 7900 2650
 Connection ~ 5500 2650
 Wire Wire Line
@@
 Wire Wire Line
 	7650 1950 7900 1950
-Connection ~ 3650 1300
-Wire Wire Line
-	3250 2250 3250 2950
+Connection ~ 3600 1300
+Wire Wire Line
+	3200 2250 3200 2950
 Wire Wire Line
 	6850 2150 6500 2150
@@
 	6500 2150 6500 2950
 Wire Wire Line
-	3550 1300 3650 1300
-Wire Wire Line
-	3650 1300 4500 1300
+	3500 1300 3600 1300
+Wire Wire Line
+	3600 1300 4500 1300
 Wire Wire Line
 	4500 1300 4750 1300
@@
 	5900 1300 6550 1300
 Wire Wire Line
-	2800 1300 3250 1300
-Wire Wire Line
-	3250 1300 3350 1300
+	2800 1300 3200 1300
+Wire Wire Line
+	3200 1300 3300 1300
 Wire Wire Line
 	2050 1300 2300 1300
@@
 	2050 2350 2050 2650
 Wire Wire Line
-	3250 1050 3250 1300
-Wire Wire Line
-	3250 1300 3250 1450
-Connection ~ 3250 1300
-Wire Wire Line
-	3650 1300 3650 1300
+	3200 1050 3200 1300
+Wire Wire Line
+	3200 1300 3200 1450
+Connection ~ 3200 1300
+Wire Wire Line
+	3600 1300 3600 1300
 Wire Wire Line
 	4500 1300 4500 1550
@@
 	5150 2100 5150 2150
 Connection ~ 5150 2100
-Connection ~ 7650 2650
 Connection ~ 6850 2650
 Connection ~ 6850 2150
 Wire Wire Line
-	2550 1750 2550 2100
-Wire Wire Line
-	2550 2500 2550 2650
-Connection ~ 2550 2650
-Wire Wire Line
 	4000 2650 4000 1850
 Wire Wire Line
-	3550 2250 3550 2250
-Wire Wire Line
-	3250 2950 2950 2950
+	3200 2950 2850 2950
 Wire Wire Line
 	6500 2950 6400 2950
@@
 PanelVoltageSense+
 Wire Wire Line
-	2950 1050 3250 1050
-Text GLabel 2950 2800 0    60   Output ~ 0
+	2950 1050 3200 1050
+Text GLabel 2850 2800 0    60   Output ~ 0
 PanelVoltageSense-
 Wire Wire Line
-	2950 2800 3150 2800
-Wire Wire Line
-	3150 2800 3150 2650
-Connection ~ 3150 2650
+	2850 2800 3000 2800
+Wire Wire Line
+	3000 2800 3000 2650
+Connection ~ 3000 2650
 Connection ~ 4000 2650
 Wire Wire Line
-	4000 1850 3850 1850
+	4000 1850 3800 1850
 Wire Wire Line
 	5150 2100 5500 2100
@@
 L R R?
 U 1 1 54D78812
-P 2800 1850
-F 0 "R?" V 2880 1850 50  0000 C CNN
-F 1 "220" V 2807 1851 50  0000 C CNN
-F 2 "" V 2730 1850 30  0000 C CNN
-F 3 "" H 2800 1850 30  0000 C CNN
-	1    2800 1850
+P 2750 1850
+F 0 "R?" V 2830 1850 50  0000 C CNN
+F 1 "220" V 2757 1851 50  0000 C CNN
+F 2 "" V 2680 1850 30  0000 C CNN
+F 3 "" H 2750 1850 30  0000 C CNN
+	1    2750 1850
 	0    1    1    0
 $EndComp
 Wire Wire Line
-	3650 1450 3650 1300
-Wire Wire Line
-	3550 1450 3550 1300
-Wire Wire Line
-	3350 1300 3350 1450
+	3600 1450 3600 1300
+Wire Wire Line
+	3500 1450 3500 1300
+Wire Wire Line
+	3300 1300 3300 1450
+Wire Wire Line
+	3000 2250 3000 1850
+Wire Wire Line
+	2500 1850 2500 1700
+Connection ~ 3500 2650
+Connection ~ 3000 1850
 $EndSCHEMATC

Commit message: mosfet power switch described
Parts:
- Q1: renamed from Q?; value MOS_N -> PSMN0R9-30YLD
- R4: renamed from R?; value R -> 1k
- gave numbers to parts that had none: 16
Connections:
- wire segments 55 -> 38
Changed lines of the file:
@@
 LIBS:relays
 LIBS:sensors
+LIBS:nxp_armmcu
 LIBS:sunpowered-cache
 EELAYER 25 0
@@
 $EndDescr
 $Comp
-L ZENER D?
+L ZENER D2
 U 1 1 54D52D0F
 P 5150 1750
-F 0 "D?" V 5150 1850 50  0000 C CNN
+F 0 "D2" V 5150 1850 50  0000 C CNN
 F 1 "24V" V 5050 1850 50  0000 C CNN
 F 2 "" H 5150 1750 60  0000 C CNN
@@
 $EndComp
 $Comp
-L CONN_01X01 P?
+L CONN_01X01 P1
 U 1 1 54D531B0
 P 850 1950
-F 0 "P?" H 850 2050 50  0000 C CNN
+F 0 "P1" H 850 2050 50  0000 C CNN
 F 1 "CONN_01X01" V 950 1950 50  0001 C CNN
 F 2 "" H 850 1950 60  0000 C CNN
@@
 $EndComp
 $Comp
-L CONN_01X01 P?
+L CONN_01X01 P2
 U 1 1 54D531ED
 P 850 2350
-F 0 "P?" H 850 2450 50  0000 C CNN
+F 0 "P2" H 850 2450 50  0000 C CNN
 F 1 "CONN_01X01" V 950 2350 50  0001 C CNN
 F 2 "" H 850 2350 60  0000 C CNN
@@
 $EndComp
 $Comp
-L FUSE F?
+L FUSE F1
 U 1 1 54D5362E
 P 2550 1300
-F 0 "F?" H 2650 1350 50  0000 C CNN
+F 0 "F1" H 2650 1350 50  0000 C CNN
 F 1 "8A" H 2450 1250 50  0000 C CNN
 F 2 "" H 2550 1300 60  0000 C CNN
@@
 $EndComp
 $Comp
-L C C?
+L C C3
 U 1 1 54D539D0
 P 4750 2050
-F 0 "C?" H 4800 2150 50  0000 L CNN
+F 0 "C3" H 4800 2150 50  0000 L CNN
 F 1 "100n" H 4800 1950 50  0000 L CNN
 F 2 "" H 4788 1900 30  0000 C CNN
@@
 $EndComp
 $Comp
-L R R?
+L R R2
 U 1 1 54D53A8D
 P 5150 2400
-F 0 "R?" H 5250 2200 50  0000 C CNN
+F 0 "R2" H 5250 2200 50  0000 C CNN
 F 1 "1k" V 5157 2401 50  0000 C CNN
 F 2 "" V 5080 2400 30  0000 C CNN
@@
 $EndComp
 $Comp
-L C C?
+L C C4
 U 1 1 54D53D1F
 P 5500 2450
-F 0 "C?" H 5550 2550 50  0000 L CNN
+F 0 "C4" H 5550 2550 50  0000 L CNN
 F 1 "47n" H 5550 2350 50  0000 L CNN
 F 2 "" H 5538 2300 30  0000 C CNN
@@
 $EndComp
 $Comp
-L THYRISTOR T?
+L THYRISTOR T1
 U 1 1 54D53E05
 P 5900 2000
-F 0 "T?" V 5900 2100 50  0000 C CNN
+F 0 "T1" V 5900 2100 50  0000 C CNN
 F 1 "12A" V 5900 1850 50  0000 C CNN
 F 2 "" H 5900 2000 60  0000 C CNN
@@
 $EndComp
 $Comp
-L DIODESCH D?
+L DIODESCH D3
 U 1 1 54D53FCE
 P 6500 1300
-F 0 "D?" H 6500 1400 50  0000 C CNN
+F 0 "D3" H 6500 1400 50  0000 C CNN
 F 1 "12A" H 6500 1200 50  0000 C CNN
 F 2 "" H 6500 1300 60  0000 C CNN
@@
 $EndComp
 $Comp
-L ZENER D?
+L ZENER D1
 U 1 1 54D5E43B
 P 4500 1750
-F 0 "D?" V 4500 1850 50  0000 C CNN
+F 0 "D1" V 4500 1850 50  0000 C CNN
 F 1 "23V" V 4400 1850 50  0000 C CNN
 F 2 "" H 4500 1750 60  0000 C CNN
@@
 $EndComp
 $Comp
-L MOS_N Q?
+L MOS_N Q1
 U 1 1 54D70F3D
 P 7550 2150
-F 0 "Q?" H 7560 2320 50  0000 R CNN
-F 1 "MOS_N" H 7500 2000 50  0000 R CNN
+F 0 "Q1" H 7500 2000 50  0000 R CNN
+F 1 "PSMN0R9-30YLD" H 8350 2200 50  0000 R CNN
 F 2 "" H 7550 2150 60  0000 C CNN
-F 3 "" H 7550 2150 60  0000 C CNN
+F 3 "http://www.nxp.com/documents/data_sheet/PSMN0R9-30YLD.pdf" H 7550 2150 60  0001 C CNN
 	1    7550 2150
 	1    0    0    -1
 $EndComp
 $Comp
-L R R?
+L R R3
 U 1 1 54D70FF3
 P 6850 2400
-F 0 "R?" V 6930 2400 50  0000 C CNN
+F 0 "R3" H 6950 2300 50  0000 C CNN
 F 1 "10k" V 6857 2401 50  0000 C CNN
 F 2 "" V 6780 2400 30  0000 C CNN
@@
 L GND #PWR01
 U 1 1 54D712EB
-P 7900 1950
-F 0 "#PWR01" H 7900 1700 60  0001 C CNN
-F 1 "GND" H 7900 1800 60  0000 C CNN
-F 2 "" H 7900 1950 60  0000 C CNN
-F 3 "" H 7900 1950 60  0000 C CNN
-	1    7900 1950
+P 7900 1650
+F 0 "#PWR01" H 7900 1400 60  0001 C CNN
+F 1 "GND" H 7900 1500 60  0000 C CNN
+F 2 "" H 7900 1650 60  0000 C CNN
+F 3 "" H 7900 1650 60  0000 C CNN
+	1    7900 1650
 	1    0    0    -1
 $EndComp
@@
 $EndComp
 $Comp
-L R R?
+L R R4
 U 1 1 54D7146D
 P 7100 2150
-F 0 "R?" V 7180 2150 50  0000 C CNN
-F 1 "R" V 7107 2151 50  0000 C CNN
+F 0 "R4" V 7000 2150 50  0000 C CNN
+F 1 "1k" V 7107 2151 50  0000 C CNN
 F 2 "" V 7030 2150 30  0000 C CNN
 F 3 "" H 7100 2150 30  0000 C CNN
@@
 $EndComp
 $Comp
-L ACS713ELCTR-30A-T IC?
+L ACS713ELCTR-30A-T IC1
 U 1 1 54D71B52
 P 3400 1850
-F 0 "IC?" V 3650 1400 50  0000 L CNN
+F 0 "IC1" V 3650 1400 50  0000 L CNN
 F 1 "ACS713" V 3250 1200 50  0000 L CNN
 F 2 "Housings_SOIC:SOIC-8_3.9x4.9mm_Pitch1.27mm" H 3400 1850 50  0001 C CIN
@@
 $EndComp
 $Comp
-L C C?
+L C C1
 U 1 1 54D74223
 P 3000 2450
-F 0 "C?" H 2850 2550 50  0000 L CNN
+F 0 "C1" H 2850 2550 50  0000 L CNN
 F 1 "0.1u" H 2800 2350 50  0000 L CNN
 F 2 "" H 3038 2300 30  0000 C CNN
@@
 $EndComp
 $Comp
-L DPST SW?
+L DPST SW1
 U 1 1 54D5CEC6
 P 1550 2150
-F 0 "SW?" H 1850 2200 50  0000 C CNN
+F 0 "SW1" H 1850 2200 50  0000 C CNN
 F 1 "DPST" H 1850 2100 50  0001 C CNN
 F 2 "" H 1550 2150 60  0000 C CNN
@@
 $EndComp
 $Comp
-L C C?
+L C C2
 U 1 1 54D76924
 P 3500 2450
-F 0 "C?" H 3550 2550 50  0000 L CNN
+F 0 "C2" H 3550 2550 50  0000 L CNN
 F 1 "47n" H 3550 2350 50  0000 L CNN
 F 2 "" H 3538 2300 30  0000 C CNN
@@
 Connection ~ 5150 2650
 Wire Wire Line
-	2050 2650 3000 2650
-Wire Wire Line
-	3000 2650 3050 2650
-Wire Wire Line
-	3000 2650 3500 2650
-Wire Wire Line
-	3500 2650 4000 2650
-Wire Wire Line
-	4000 2650 4500 2650
-Wire Wire Line
-	4500 2650 4750 2650
-Wire Wire Line
-	4750 2650 5150 2650
-Wire Wire Line
-	5150 2650 5500 2650
-Wire Wire Line
-	5500 2650 5900 2650
-Wire Wire Line
-	5900 2650 6850 2650
-Wire Wire Line
-	6850 2650 7650 2650
+	2050 2650 3050 2650
+Wire Wire Line
+	3000 2650 7650 2650
 Connection ~ 5500 2650
 Wire Wire Line
@@
 Wire Wire Line
 	6700 1300 7900 1300
-Wire Wire Line
-	7650 2650 7650 2300
 Connection ~ 4500 1300
 Wire Wire Line
-	7650 1950 7900 1950
+	7650 1650 7900 1650
 Connection ~ 3600 1300
 Wire Wire Line
@@
 	6500 2150 6500 2950
 Wire Wire Line
-	3500 1300 3600 1300
-Wire Wire Line
-	3600 1300 4500 1300
-Wire Wire Line
-	4500 1300 4750 1300
-Wire Wire Line
-	4750 1300 5150 1300
-Wire Wire Line
-	5150 1300 5900 1300
-Wire Wire Line
-	5900 1300 6550 1300
-Wire Wire Line
-	2800 1300 3200 1300
-Wire Wire Line
-	3200 1300 3300 1300
+	3500 1300 6550 1300
+Wire Wire Line
+	2800 1300 3300 1300
 Wire Wire Line
 	2050 1300 2300 1300
@@
 	2050 2350 2050 2650
 Wire Wire Line
-	3200 1050 3200 1300
-Wire Wire Line
-	3200 1300 3200 1450
+	3200 1050 3200 1450
 Connection ~ 3200 1300
 Wire Wire Line
@@
 	5150 1300 5150 1550
 Wire Wire Line
-	5150 1950 5150 2100
-Wire Wire Line
-	5150 2100 5150 2150
+	5150 1950 5150 2150
 Connection ~ 5150 2100
 Connection ~ 6850 2650
@@
 	4000 1850 3800 1850
 Wire Wire Line
-	5150 2100 5500 2100
-Wire Wire Line
-	5500 2100 5750 2100
+	5150 2100 5750 2100
 Wire Wire Line
 	5500 2250 5500 2100
 Connection ~ 5500 2100
 $Comp
-L R R?
+L R R1
 U 1 1 54D78812
 P 2750 1850
-F 0 "R?" V 2830 1850 50  0000 C CNN
+F 0 "R1" V 2830 1850 50  0000 C CNN
 F 1 "220" V 2757 1851 50  0000 C CNN
 F 2 "" V 2680 1850 30  0000 C CNN
@@
 Connection ~ 3500 2650
 Connection ~ 3000 1850
+Wire Wire Line
+	7650 1650 7650 1950
+Wire Wire Line
+	7650 2650 7650 2350
 $EndSCHEMATC

Commit message: power on soft-switch now features always-on capability. Added connector with all measurements
Parts:
- removed P1, P2: CONN_01X01, symbol CONN_01X01
- added C5: 4700u, symbol CP2
- added JP1: JUMPER3, symbol JUMPER3
- added P1: CONN_01X02, symbol CONN_01X02
- added P2: CONN_02X04, symbol CONN_02X04
- added R5: 5k, symbol R
- D2: Note OV protection -> (none)
Connections:
- net labels added: +5V, GNDD
- net labels removed: +5P
- wire segments 38 -> 62
Other:
- note added: "Always On"
- note added: "External"
- note added: "Input measurements"
- note added: "Overvoltage protection"
- note added: "Power on soft switch"
- moved on the sheet: C1, C2, C3, C4, D1, D2, D3, F1, IC1, Q1, R1, R2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
