File: electronics/sunpowered.kicad_pcb (KiCad board)
At the start: 2 copper layers, 0 parts

Commit message: all footprints added, started layout
Parts:
- added C1: 4700u, Capacitors_ThroughHole:Capacitor5x11RM2.5, F.Cu at (135.9, 120.7)
- added C2: 100n, Capacitors_SMD:C_0603_HandSoldering, F.Cu at (144.8, 121.9)
- added C3: 47n, Capacitors_SMD:C_0603_HandSoldering, F.Cu at (146.1, 111.8)
- added C4: 100n, Capacitors_SMD:C_0603_HandSoldering, F.Cu at (156.2, 109.2)
- added C5: 47n, Capacitors_SMD:C_0603_HandSoldering, F.Cu at (148.5, 105.0)
- added D1: 24V, Diodes_SMD:Diode-SMC_Handsoldering, F.Cu at (175.3, 118.1)
- added D2: 12A, cyplo's:TO277A, F.Cu at (158.8, 116.8)
- added F1: 8A, Fuse_Holders_and_Fuses:Fuseholder5x20_horiz_open_universal_Type-III, F.Cu at (141.0, 101.6)
- added IC1: ACS713, Housings_SOIC:SOIC-8_3.9x4.9mm_Pitch1.27mm, F.Cu at (161.3, 99.1)
- added JP1: JUMPER3, Pin_Headers:Pin_Header_Straight_1x03, F.Cu at (189.2, 97.8)
- added P1: CONN_01X02, Terminal_Blocks:TerminalBlock_WAGO-236_2Stift_RM5mm_2pol, F.Cu at (120.7, 105.4)
- added P2: CONN_02X04, Pin_Headers:Pin_Header_Straight_2x04, F.Cu at (191.8, 119.4)
- added P3: CONN_01X02, Terminal_Blocks:TerminalBlock_WAGO-236_2Stift_RM5mm_2pol, F.Cu at (198.1, 102.9)
- added Q1: PSMN0R9-30YLD, cyplo's:LFPAK56, F.Cu at (186.7, 113.0)
- added R1: 330, Resistors_SMD:R_0603_HandSoldering, F.Cu at (148.5, 105.0)
- added R2: 1k, Resistors_SMD:R_0603_HandSoldering, F.Cu at (148.5, 105.0)
- added R3: 5k, Resistors_SMD:R_0603_HandSoldering, F.Cu at (148.6, 115.6)
- added R4: 10k, Resistors_SMD:R_0603_HandSoldering, F.Cu at (148.5, 105.0)
- added R5: 1k, Resistors_SMD:R_0603_HandSoldering, F.Cu at (161.3, 108.0)
- added T1: 12A, Transistors_SMD:sot428, F.Cu at (181.6, 102.9)
Other:
- rule pad_to_mask_clearance: 0 -> 0.2
