File: electronics/input_board.sch (KiCad schematic (older format))
At the start: 20 parts

Commit message: wires that went missing after copying from sheet to sheet added
Parts:
- gave numbers to parts that had none: 20
Connections:
- net labels added: DigitalGround
- wire segments 52 -> 61
Changed lines of the file:
@@
 $EndDescr
 $Comp
-L ZENER D?
+L ZENER D1
 U 1 1 55E0D9D5
 P 5750 1750
-F 0 "D?" V 5750 1850 50  0000 C CNN
+F 0 "D1" V 5750 1850 50  0000 C CNN
 F 1 "24V" V 5650 1850 50  0000 C CNN
 F 2 "Diodes_SMD:Diode-SMC_Handsoldering" H 5750 1750 60  0001 C CNN
@@
 F 4 "~" V 5850 1400 39  0000 C CNN "Note"
 	1    5750 1750
-	0    -1   -1   0
-$EndComp
-$Comp
-L FUSE F?
+	0    1    1    0
+$EndComp
+$Comp
+L FUSE F1
 U 1 1 55E0D9DC
 P 3150 1300
-F 0 "F?" H 3250 1350 50  0000 C CNN
+F 0 "F1" H 3250 1350 50  0000 C CNN
 F 1 "8A" H 3050 1250 50  0000 C CNN
 F 2 "Fuse_Holders_and_Fuses:Fuseholder5x20_horiz_open_universal_Type-III" H 3150 1300 60  0001 C CNN
@@
 $EndComp
 $Comp
-L C C?
+L C C4
 U 1 1 55E0D9E3
 P 5350 2050
-F 0 "C?" H 5400 2150 50  0000 L CNN
+F 0 "C4" H 5400 2150 50  0000 L CNN
 F 1 "100n" H 5400 1950 50  0000 L CNN
 F 2 "Capacitors_SMD:C_0603_HandSoldering" H 5388 1900 30  0001 C CNN
@@
 $EndComp
 $Comp
-L R R?
+L R R2
 U 1 1 55E0D9EA
 P 5750 2400
-F 0 "R?" H 5850 2200 50  0000 C CNN
+F 0 "R2" H 5850 2200 50  0000 C CNN
 F 1 "1k" V 5757 2401 50  0000 C CNN
 F 2 "Resistors_SMD:R_0603_HandSoldering" V 5680 2400 30  0001 C CNN
@@
 $EndComp
 $Comp
-L C C?
+L C C5
 U 1 1 55E0D9F1
 P 6100 2450
-F 0 "C?" H 6150 2550 50  0000 L CNN
+F 0 "C5" H 6150 2550 50  0000 L CNN
 F 1 "47n" H 6150 2350 50  0000 L CNN
 F 2 "Capacitors_SMD:C_0603_HandSoldering" H 6138 2300 30  0001 C CNN
@@
 $EndComp
 $Comp
-L THYRISTOR T?
+L THYRISTOR T1
 U 1 1 55E0D9F8
 P 6500 2000
-F 0 "T?" V 6500 2100 50  0000 C CNN
+F 0 "T1" V 6500 2100 50  0000 C CNN
 F 1 "12A" V 6500 1850 50  0000 C CNN
 F 2 "cyplo's:sot428" H 6500 2000 60  0001 C CNN
 F 3 "http://www.nxp.com/documents/data_sheet/BT151S_SER_L_R.pdf" H 6500 2000 60  0001 C CNN
 	1    6500 2000
-	0    -1   1    0
-$EndComp
-$Comp
-L DIODESCH D?
+	0    -1   -1   0
+$EndComp
+$Comp
+L DIODESCH D2
 U 1 1 55E0D9FF
 P 7050 1300
-F 0 "D?" H 7050 1400 50  0000 C CNN
+F 0 "D2" H 7050 1400 50  0000 C CNN
 F 1 "12A" H 7050 1200 50  0000 C CNN
 F 2 "cyplo's:TO277A" H 7050 1300 60  0001 C CNN
@@
 $EndComp
 $Comp
-L MOS_N Q?
+L MOS_N Q1
 U 1 1 55E0DA06
 P 8150 2150
-F 0 "Q?" H 8100 2000 50  0000 R CNN
+F 0 "Q1" H 8100 2000 50  0000 R CNN
 F 1 "PSMN0R9-30YLD" V 8350 2400 50  0000 R CNN
 F 2 "cyplo's:LFPAK56" H 8150 2150 60  0001 C CNN
@@
 $EndComp
 $Comp
-L R R?
+L R R4
 U 1 1 55E0DA0D
 P 7450 2400
-F 0 "R?" H 7550 2300 50  0000 C CNN
+F 0 "R4" H 7550 2300 50  0000 C CNN
 F 1 "10k" V 7457 2401 50  0000 C CNN
 F 2 "Resistors_SMD:R_0603_HandSoldering" V 7380 2400 30  0001 C CNN
@@
 $EndComp
 $Comp
-L R R?
+L R R5
 U 1 1 55E0DA14
 P 7700 2150
-F 0 "R?" V 7600 2150 50  0000 C CNN
+F 0 "R5" V 7600 2150 50  0000 C CNN
 F 1 "1k" V 7707 2151 50  0000 C CNN
 F 2 "Resistors_SMD:R_0603_HandSoldering" V 7630 2150 30  0001 C CNN
@@
 $EndComp
 $Comp
-L C C?
+L C C2
 U 1 1 55E0DA1B
 P 3450 2000
-F 0 "C?" H 3300 1900 50  0000 L CNN
+F 0 "C2" H 3300 1900 50  0000 L CNN
 F 1 "100n" H 3250 2100 50  0000 L CNN
 F 2 "Capacitors_SMD:C_0603_HandSoldering" H 3488 1850 30  0001 C CNN
@@
 $EndComp
 $Comp
-L C C?
+L C C3
 U 1 1 55E0DA22
 P 4300 2150
-F 0 "C?" V 4350 2200 50  0000 L CNN
+F 0 "C3" V 4350 2200 50  0000 L CNN
 F 1 "47n" V 4350 1950 50  0000 L CNN
 F 2 "Capacitors_SMD:C_0603_HandSoldering" H 4338 2000 30  0001 C CNN
@@
 PanelVoltageSense-
 $Comp
-L R R?
+L R R1
 U 1 1 55E0DA2C
 P 3100 1700
-F 0 "R?" V 3180 1700 50  0000 C CNN
+F 0 "R1" V 3180 1700 50  0000 C CNN
 F 1 "330" V 3107 1701 50  0000 C CNN
 F 2 "Resistors_SMD:R_0603_HandSoldering" V 3030 1700 30  0001 C CNN
@@
 $EndComp
 $Comp
-L ACS713ELCTR-30A-T IC?
+L ACS713ELCTR-30A-T IC1
 U 1 1 55E0DA34
 P 4000 1700
-F 0 "IC?" V 4250 1250 50  0000 L CNN
+F 0 "IC1" V 4250 1250 50  0000 L CNN
 F 1 "ACS713" V 3850 1050 50  0000 L CNN
 F 2 "Housings_SOIC:SOIC-8_3.9x4.9mm_Pitch1.27mm" H 4000 1700 50  0001 C CIN
@@
 Power on soft switch
 $Comp
-L CONN_01X02 P?
+L CONN_01X02 P1
 U 1 1 55E0DA3E
 P 1450 2150
-F 0 "P?" H 1450 2300 50  0000 C CNN
+F 0 "P1" H 1450 2300 50  0000 C CNN
 F 1 "CONN_01X02" V 1550 2150 50  0000 C CNN
 F 2 "Terminal_Blocks:TerminalBlock_WAGO-236_2Stift_RM5mm_2pol" H 1450 2150 60  0001 C CNN
@@
 $EndComp
 $Comp
-L JUMPER3 JP?
+L JUMPER3 JP1
 U 1 1 55E0DA45
 P 7250 2150
-F 0 "JP?" H 7300 2050 50  0000 L CNN
+F 0 "JP1" H 7300 2050 50  0000 L CNN
 F 1 "JUMPER3" H 7250 2250 50  0001 C BNN
 F 2 "Pin_Headers:Pin_Header_Straight_1x03" H 7250 2150 60  0001 C CNN
@@
 $EndComp
 $Comp
-L GNDD #PWR?
+L GNDD #PWR5
 U 1 1 55E0DA4C
 P 3450 2300
-F 0 "#PWR?" H 3450 2050 60  0001 C CNN
+F 0 "#PWR5" H 3450 2050 60  0001 C CNN
 F 1 "GNDD" H 3450 2150 60  0000 C CNN
 F 2 "" H 3450 2300 60  0000 C CNN
@@
 $EndComp
 $Comp
-L R R?
+L R R3
 U 1 1 55E0DA52
 P 7250 1550
-F 0 "R?" H 7350 1550 50  0000 C CNN
+F 0 "R3" H 7350 1550 50  0000 C CNN
 F 1 "5k" V 7257 1551 50  0000 C CNN
 F 2 "Resistors_SMD:R_0603_HandSoldering" V 7180 1550 30  0001 C CNN
@@
 PowerOn
 $Comp
-L GNDD #PWR?
+L GNDD #PWR6
 U 1 1 55E0DA5C
 P 4600 2350
-F 0 "#PWR?" H 4600 2100 60  0001 C CNN
+F 0 "#PWR6" H 4600 2100 60  0001 C CNN
 F 1 "GNDD" H 4600 2200 60  0000 C CNN
 F 2 "" H 4600 2350 60  0000 C CNN
@@
 $EndComp
 $Comp
-L CONN_01X02 P?
+L CONN_01X02 P3
 U 1 1 55E0DA62
 P 8700 1350
-F 0 "P?" H 8700 1500 50  0000 C CNN
+F 0 "P3" H 8700 1500 50  0000 C CNN
 F 1 "CONN_01X02" V 8800 1350 50  0000 C CNN
 F 2 "Terminal_Blocks:TerminalBlock_WAGO-236_2Stift_RM5mm_2pol" H 8700 1350 60  0001 C CNN
@@
 $EndComp
 $Comp
-L PWR_FLAG #FLG?
+L PWR_FLAG #FLG4
 U 1 1 55E0DA69
 P 4200 1300
-F 0 "#FLG?" H 4200 1395 30  0001 C CNN
+F 0 "#FLG4" H 4200 1395 30  0001 C CNN
 F 1 "PWR_FLAG" H 4200 1480 30  0001 C CNN
 F 2 "" H 4200 1300 60  0000 C CNN
@@
 $EndComp
 $Comp
-L +5V #PWR?
+L +5V #PWR2
 U 1 1 55E0DA6F
 P 2850 1600
-F 0 "#PWR?" H 2850 1450 60  0001 C CNN
+F 0 "#PWR2" H 2850 1450 60  0001 C CNN
 F 1 "+5V" H 2850 1740 60  0000 C CNN
 F 2 "" H 2850 1600 60  0000 C CNN
@@
 Connection ~ 5750 2650
 Connection ~ 6100 2650
-Wire Wire Line
-	6500 1300 6500 1800
 Connection ~ 6500 1300
-Wire Wire Line
-	6500 2650 6500 2200
 Connection ~ 6500 2650
 Wire Wire Line
-	5350 2650 5350 2250
+	5350 2200 5350 2650
 Connection ~ 5350 2650
 Wire Wire Line
-	5350 1300 5350 1850
+	5350 1300 5350 1900
 Connection ~ 5350 1300
 Wire Wire Line
@@
 	3800 2100 3800 3000
 Wire Wire Line
-	7450 2150 7350 2150
+	7350 2150 7550 2150
 Wire Wire Line
 	3400 1300 3900 1300
@@
 	5750 1300 5750 1550
 Wire Wire Line
-	5750 1950 5750 2150
+	5750 1950 5750 2250
 Connection ~ 5750 2100
 Connection ~ 7450 2650
@@
 	3550 1050 3800 1050
 Wire Wire Line
-	5750 2100 6350 2100
-Wire Wire Line
-	6100 2250 6100 2100
+	6100 2100 6100 2300
 Connection ~ 6100 2100
 Wire Wire Line
@@
 	1650 2650 8250 2650
 Wire Wire Line
-	7250 1800 7250 1900
+	7250 1700 7250 1900
 Wire Wire Line
 	4100 2100 4100 2150
@@
 	4600 1700 4600 2350
 Wire Wire Line
-	4600 2150 4500 2150
+	4450 2150 4600 2150
 Connection ~ 4600 2150
 Wire Wire Line
@@
 	4100 1300 6850 1300
 Wire Wire Line
-	3350 1700 3600 1700
+	3250 1700 3600 1700
 Wire Wire Line
 	3450 2300 3450 2200
 Wire Wire Line
-	3450 1800 3450 1700
+	3450 1700 3450 1850
 Connection ~ 3450 1700
 Wire Wire Line
 	2850 1600 2850 1700
 $Comp
-L PWR_FLAG #FLG?
+L PWR_FLAG #FLG1
 U 1 1 55E0DAAC
 P 2650 1300
-F 0 "#FLG?" H 2650 1395 30  0001 C CNN
+F 0 "#FLG1" H 2650 1395 30  0001 C CNN
 F 1 "PWR_FLAG" H 2650 1480 30  0001 C CNN
 F 2 "" H 2650 1300 60  0000 C CNN
@@
 15mA
 $Comp
-L PWR_FLAG #FLG?
+L PWR_FLAG #FLG3
 U 1 1 55E0DAB3
 P 3450 1700
-F 0 "#FLG?" H 3450 1795 30  0001 C CNN
+F 0 "#FLG3" H 3450 1795 30  0001 C CNN
 F 1 "PWR_FLAG" H 3450 1880 30  0001 C CNN
 F 2 "" H 3450 1700 60  0000 C CNN
@@
 PanelVoltageSense+
 $Comp
-L CP2 C?
+L CP2 C1
 U 1 1 55E0DF59
 P 3050 4100
-F 0 "C?" H 2850 4100 50  0000 L CNN
+F 0 "C1" H 2850 4100 50  0000 L CNN
 F 1 "4700u" H 3150 4100 50  0000 L CNN
 F 2 "Capacitors_ThroughHole:Capacitor5x11RM2.5" H 3088 3950 30  0001 C CNN
@@
 $EndComp
 $Comp
-L +5V #PWR?
+L +5V #PWR4
 U 1 1 55E0DF60
 P 3350 3900
-F 0 "#PWR?" H 3350 3750 60  0001 C CNN
+F 0 "#PWR4" H 3350 3750 60  0001 C CNN
 F 1 "+5V" H 3350 4040 60  0000 C CNN
 F 2 "" H 3350 3900 60  0000 C CNN
@@
 	2200 3900 3350 3900
 $Comp
-L PWR_FLAG #FLG?
+L PWR_FLAG #FLG2
 U 1 1 55E0DF67
 P 3050 3900
-F 0 "#FLG?" H 3050 3995 30  0001 C CNN
+F 0 "#FLG2" H 3050 3995 30  0001 C CNN
 F 1 "PWR_FLAG" H 3050 4080 30  0001 C CNN
 F 2 "" H 3050 3900 60  0000 C CNN
@@
 Connection ~ 3050 3900
 $Comp
-L GNDD #PWR?
+L GNDD #PWR3
 U 1 1 55E0DF6E
 P 3050 4300
-F 0 "#PWR?" H 3050 4050 60  0001 C CNN
+F 0 "#PWR3" H 3050 4050 60  0001 C CNN
 F 1 "GNDD" H 3050 4150 60  0000 C CNN
 F 2 "" H 3050 4300 60  0000 C CNN
@@
 CurrentSensorVoltageSense
 $Comp
-L CONN_02X05 P?
+L CONN_02X05 P2
 U 1 1 55E0DF75
 P 1950 4100
-F 0 "P?" H 1950 4400 50  0000 C CNN
+F 0 "P2" H 1950 4400 50  0000 C CNN
 F 1 "CONN_02X05" H 1950 4500 50  0000 C CNN
 F 2 "" H 1950 2900 60  0000 C CNN
@@
 Connection ~ 1700 4000
 $Comp
-L GNDD #PWR?
+L GNDD #PWR1
 U 1 1 55E0DF80
 P 1700 4450
-F 0 "#PWR?" H 1700 4200 60  0001 C CNN
+F 0 "#PWR1" H 1700 4200 60  0001 C CNN
 F 1 "GNDD" H 1700 4300 60  0000 C CNN
 F 2 "" H 1700 4450 60  0000 C CNN
@@
 Wire Wire Line
 	2500 4200 2500 4650
+Text GLabel 1350 4300 0    60   BiDi ~ 0
+DigitalGround
+Wire Wire Line
+	1350 4300 1700 4300
+Wire Wire Line
+	7950 2150 7850 2150
+Wire Wire Line
+	7450 2150 7450 2250
+Wire Wire Line
+	7450 2550 7450 2650
+Wire Wire Line
+	7250 1400 7250 1300
+Wire Wire Line
+	6100 2600 6100 2650
+Wire Wire Line
+	5750 2550 5750 2650
+Wire Wire Line
+	4100 2150 4150 2150
+Wire Wire Line
+	2850 1700 2950 1700
+Wire Wire Line
+	6500 2650 6500 2200
+Wire Wire Line
+	5750 2100 6400 2100
+Wire Wire Line
+	6500 1800 6500 1300
 $EndSCHEMATC

Commit message: input baord: initial component placement
Parts:
- C1: footprint Capacitors_ThroughHole:Capacitor5x11RM2.5 -> Capacitors_ThroughHole:C_Radial_D13_L25_P5
- P2: footprint (none) -> Pin_Headers:Pin_Header_Straight_2x05
Connections:
- wire segments 61 -> 62
Changed lines of the file:
@@
 $EndComp
 $Comp
-L GNDD #PWR5
+L GNDD #PWR01
 U 1 1 55E0DA4C
 P 3450 2300
-F 0 "#PWR5" H 3450 2050 60  0001 C CNN
+F 0 "#PWR01" H 3450 2050 60  0001 C CNN
 F 1 "GNDD" H 3450 2150 60  0000 C CNN
 F 2 "" H 3450 2300 60  0000 C CNN
@@
 PowerOn
 $Comp
-L GNDD #PWR6
+L GNDD #PWR02
 U 1 1 55E0DA5C
 P 4600 2350
-F 0 "#PWR6" H 4600 2100 60  0001 C CNN
+F 0 "#PWR02" H 4600 2100 60  0001 C CNN
 F 1 "GNDD" H 4600 2200 60  0000 C CNN
 F 2 "" H 4600 2350 60  0000 C CNN
@@
 $EndComp
 $Comp
-L PWR_FLAG #FLG4
+L PWR_FLAG #FLG03
 U 1 1 55E0DA69
 P 4200 1300
-F 0 "#FLG4" H 4200 1395 30  0001 C CNN
+F 0 "#FLG03" H 4200 1395 30  0001 C CNN
 F 1 "PWR_FLAG" H 4200 1480 30  0001 C CNN
 F 2 "" H 4200 1300 60  0000 C CNN
@@
 $EndComp
 $Comp
-L +5V #PWR2
+L +5V #PWR04
 U 1 1 55E0DA6F
 P 2850 1600
-F 0 "#PWR2" H 2850 1450 60  0001 C CNN
+F 0 "#PWR04" H 2850 1450 60  0001 C CNN
 F 1 "+5V" H 2850 1740 60  0000 C CNN
 F 2 "" H 2850 1600 60  0000 C CNN
@@
 	2850 1600 2850 1700
 $Comp
-L PWR_FLAG #FLG1
+L PWR_FLAG #FLG05
 U 1 1 55E0DAAC
 P 2650 1300
-F 0 "#FLG1" H 2650 1395 30  0001 C CNN
+F 0 "#FLG05" H 2650 1395 30  0001 C CNN
 F 1 "PWR_FLAG" H 2650 1480 30  0001 C CNN
 F 2 "" H 2650 1300 60  0000 C CNN
@@
 15mA
 $Comp
-L PWR_FLAG #FLG3
+L PWR_FLAG #FLG06
 U 1 1 55E0DAB3
 P 3450 1700
-F 0 "#FLG3" H 3450 1795 30  0001 C CNN
+F 0 "#FLG06" H 3450 1795 30  0001 C CNN
 F 1 "PWR_FLAG" H 3450 1880 30  0001 C CNN
 F 2 "" H 3450 1700 60  0000 C CNN
@@
 F 0 "C1" H 2850 4100 50  0000 L CNN
 F 1 "4700u" H 3150 4100 50  0000 L CNN
-F 2 "Capacitors_ThroughHole:Capacitor5x11RM2.5" H 3088 3950 30  0001 C CNN
+F 2 "Capacitors_ThroughHole:C_Radial_D13_L25_P5" H 3088 3950 30  0001 C CNN
 F 3 "" H 3050 4100 60  0000 C CNN
 	1    3050 4100
@@
 $EndComp
 $Comp
-L +5V #PWR4
+L +5V #PWR07
 U 1 1 55E0DF60
 P 3350 3900
-F 0 "#PWR4" H 3350 3750 60  0001 C CNN
+F 0 "#PWR07" H 3350 3750 60  0001 C CNN
 F 1 "+5V" H 3350 4040 60  0000 C CNN
 F 2 "" H 3350 3900 60  0000 C CNN
@@
 	2200 3900 3350 3900
 $Comp
-L PWR_FLAG #FLG2
+L PWR_FLAG #FLG08
 U 1 1 55E0DF67
 P 3050 3900
-F 0 "#FLG2" H 3050 3995 30  0001 C CNN
+F 0 "#FLG08" H 3050 3995 30  0001 C CNN
 F 1 "PWR_FLAG" H 3050 4080 30  0001 C CNN
 F 2 "" H 3050 3900 60  0000 C CNN
@@
 Connection ~ 3050 3900
 $Comp
-L GNDD #PWR3
+L GNDD #PWR09
 U 1 1 55E0DF6E
 P 3050 4300
-F 0 "#PWR3" H 3050 4050 60  0001 C CNN
+F 0 "#PWR09" H 3050 4050 60  0001 C CNN
 F 1 "GNDD" H 3050 4150 60  0000 C CNN
 F 2 "" H 3050 4300 60  0000 C CNN
@@
 P 1950 4100
 F 0 "P2" H 1950 4400 50  0000 C CNN
-F 1 "CONN_02X05" H 1950 4500 50  0000 C CNN
-F 2 "" H 1950 2900 60  0000 C CNN
+F 1 "CONN_02X05" H 1800 4500 50  0000 C CNN
+F 2 "Pin_Headers:Pin_Header_Straight_2x05" H 1950 2900 60  0000 C CNN
 F 3 "" H 1950 2900 60  0000 C CNN
 	1    1950 4100
@@
 Connection ~ 1700 4000
 $Comp
-L GNDD #PWR1
+L GNDD #PWR010
 U 1 1 55E0DF80
 P 1700 4450
-F 0 "#PWR1" H 1700 4200 60  0001 C CNN
+F 0 "#PWR010" H 1700 4200 60  0001 C CNN
 F 1 "GNDD" H 1700 4300 60  0000 C CNN
 F 2 "" H 1700 4450 60  0000 C CNN
@@
 Wire Wire Line
 	6500 1800 6500 1300
+Text GLabel 2200 3850 1    60   BiDi ~ 0
++5V
+Wire Wire Line
+	2200 3850 2200 3900
+Connection ~ 2200 3900
 $EndSCHEMATC

Commit message: Upgrade to the newest KiCad version + better caps.
Some of the component symbols got lost while upgrading to the newest KiCad,
recreated them.
Calculated better filter cap values.
Parts:
- removed C1: 4700u, Capacitors_ThroughHole:C_Radial_D13_L25_P5, symbol CP2
- removed D2: 12A, cyplo's:TO277A, symbol DIODESCH
- removed Q1: PSMN0R9-30YLD, cyplo's:LFPAK56, symbol MOS_N
- added C1: 10u, Capacitors_SMD:C_0603_HandSoldering, symbol C
- added D2: 12A, cyplo's:TO277A, symbol D_Schottky
- added Q1: Q_NMOS_SGD, cyplo's:LFPAK56, symbol Q_NMOS_SGD
Connections:
- wire segments 62 -> 64
Changed lines of the file:
@@
 LIBS:memory
 LIBS:xilinx
-LIBS:special
 LIBS:microcontrollers
 LIBS:dsp
@@
 LIBS:nxp_armmcu
 LIBS:dc-dc
-LIBS:sunpowered-cache
+LIBS:powerint
+LIBS:Power_Management
+LIBS:ab2_connectivity
+LIBS:ab2_idc
+LIBS:ab2_terminal_block
 EELAYER 25 0
 EELAYER END
@@
 $EndComp
 $Comp
-L DIODESCH D2
-U 1 1 55E0D9FF
-P 7050 1300
-F 0 "D2" H 7050 1400 50  0000 C CNN
-F 1 "12A" H 7050 1200 50  0000 C CNN
-F 2 "cyplo's:TO277A" H 7050 1300 60  0001 C CNN
-F 3 "http://www.vishay.com/docs/89094/v12p12.pdf" H 7050 1300 60  0001 C CNN
-	1    7050 1300
-	1    0    0    -1
-$EndComp
-$Comp
-L MOS_N Q1
-U 1 1 55E0DA06
-P 8150 2150
-F 0 "Q1" H 8100 2000 50  0000 R CNN
-F 1 "PSMN0R9-30YLD" V 8350 2400 50  0000 R CNN
-F 2 "cyplo's:LFPAK56" H 8150 2150 60  0001 C CNN
-F 3 "http://www.nxp.com/documents/data_sheet/PSMN0R9-30YLD.pdf" H 8150 2150 60  0001 C CNN
-	1    8150 2150
-	1    0    0    -1
-$EndComp
-$Comp
 L R R4
 U 1 1 55E0DA0D
@@
 	1650 2200 1650 2650
 Wire Wire Line
-	7250 1300 8500 1300
+	7200 1300 8500 1300
 Connection ~ 7250 1300
-Wire Wire Line
-	7250 2400 7250 3000
 Wire Wire Line
 	7250 3000 7200 3000
@@
 	4600 1700 4400 1700
 Wire Wire Line
-	4100 1300 6850 1300
+	4100 1300 6900 1300
 Wire Wire Line
 	3250 1700 3600 1700
@@
 Text GLabel 2500 4650 3    60   Input ~ 0
 PanelCurrentSense
-Text GLabel 1150 3900 2    60   Output ~ 0
+Text GLabel 1550 3900 0    60   Output ~ 0
 PowerOn
 Text GLabel 2300 4650 3    60   Input ~ 0
@@
 Text GLabel 2850 4650 3    60   Input ~ 0
 PanelVoltageSense+
-$Comp
-L CP2 C1
-U 1 1 55E0DF59
-P 3050 4100
-F 0 "C1" H 2850 4100 50  0000 L CNN
-F 1 "4700u" H 3150 4100 50  0000 L CNN
-F 2 "Capacitors_ThroughHole:C_Radial_D13_L25_P5" H 3088 3950 30  0001 C CNN
-F 3 "" H 3050 4100 60  0000 C CNN
-	1    3050 4100
-	1    0    0    -1
-$EndComp
 $Comp
 L +5V #PWR07
@@
 $EndComp
 Connection ~ 3050 3900
-$Comp
-L GNDD #PWR09
-U 1 1 55E0DF6E
-P 3050 4300
-F 0 "#PWR09" H 3050 4050 60  0001 C CNN
-F 1 "GNDD" H 3050 4150 60  0000 C CNN
-F 2 "" H 3050 4300 60  0000 C CNN
-F 3 "" H 3050 4300 60  0000 C CNN
-	1    3050 4300
-	1    0    0    -1
-$EndComp
 Text GLabel 2650 4650 3    60   Input ~ 0
 CurrentSensorVoltageSense
@@
 F 0 "P2" H 1950 4400 50  0000 C CNN
 F 1 "CONN_02X05" H 1800 4500 50  0000 C CNN
-F 2 "Pin_Headers:Pin_Header_Straight_2x05" H 1950 2900 60  0000 C CNN
+F 2 "Pin_Headers:Pin_Header_Straight_2x05" H 1950 2900 60  0001 C CNN
 F 3 "" H 1950 2900 60  0000 C CNN
 	1    1950 4100
@@
 Connection ~ 1700 4000
 $Comp
-L GNDD #PWR010
+L GNDD #PWR09
 U 1 1 55E0DF80
-P 1700 4450
-F 0 "#PWR010" H 1700 4200 60  0001 C CNN
-F 1 "GNDD" H 1700 4300 60  0000 C CNN
-F 2 "" H 1700 4450 60  0000 C CNN
-F 3 "" H 1700 4450 60  0000 C CNN
-	1    1700 4450
+P 1700 4550
+F 0 "#PWR09" H 1700 4300 60  0001 C CNN
+F 1 "GNDD" H 1700 4400 60  0000 C CNN
+F 2 "" H 1700 4550 60  0000 C CNN
+F 3 "" H 1700 4550 60  0000 C CNN
+	1    1700 4550
 	1    0    0    -1
 $EndComp
@@
 Wire Wire Line
 	2200 4000 2850 4000
-Wire Wire Line
-	1700 4000 1700 4450
-Wire Wire Line
-	1600 3900 1700 3900
 Wire Wire Line
 	2650 4100 2650 4650
@@
 	2200 3850 2200 3900
 Connection ~ 2200 3900
+$Comp
+L D_Schottky D2
+U 1 1 55EBE3EF
+P 7050 1300
+F 0 "D2" H 7050 1400 50  0000 C CNN
+F 1 "12A" H 7050 1200 50  0000 C CNN
+F 2 "cyplo's:TO277A" H 7050 1300 60  0001 C CNN
+F 3 "http://www.vishay.com/docs/89094/v12p12.pdf" H 7050 1300 60  0001 C CNN
+	1    7050 1300
+	-1   0    0    1
+$EndComp
+$Comp
+L Q_NMOS_SGD Q1
+U 1 1 55EBE70C
+P 8150 2150
+F 0 "Q1" H 8450 2200 50  0000 R CNN
+F 1 "Q_NMOS_SGD" H 8800 2100 50  0000 R CNN
+F 2 "cyplo's:LFPAK56" H 8350 2250 29  0001 C CNN
+F 3 "http://www.nxp.com/documents/data_sheet/PSMN0R9-30YLD.pdf" H 8150 2150 60  0001 C CNN
+	1    8150 2150
+	1    0    0    -1
+$EndComp
+$Comp
+L C C1
+U 1 1 55EBF3A1
+P 7900 2400
+F 0 "C1" H 7950 2500 50  0000 L CNN
+F 1 "10u" H 7950 2300 50  0000 L CNN
+F 2 "Capacitors_SMD:C_0603_HandSoldering" H 7938 2250 30  0001 C CNN
+F 3 "" H 7900 2400 60  0000 C CNN
+	1    7900 2400
+	1    0    0    -1
+$EndComp
+Wire Wire Line
+	7900 2550 7900 2650
+Connection ~ 7900 2650
+Wire Wire Line
+	7900 2250 7900 2150
+Connection ~ 7900 2150
+Wire Wire Line
+	7250 3000 7250 2400
+Wire Wire Line
+	1700 3900 1550 3900
+Wire Wire Line
+	1700 4000 1700 4550
 $EndSCHEMATC

Commit message: Added 5V 3A power supply
Connections:
- net labels added: RawGround, RawPositive
- net labels removed: DigitalGround
- wire segments 64 -> 65
Changed lines of the file:
@@
 LIBS:memory
 LIBS:xilinx
-LIBS:microcontrollers
-LIBS:dsp
-LIBS:microchip
-LIBS:analog_switches
-LIBS:motorola
-LIBS:texas
-LIBS:intel
-LIBS:audio
-LIBS:interface
-LIBS:digital-audio
-LIBS:philips
-LIBS:display
-LIBS:cypress
-LIBS:siliconi
-LIBS:opto
-LIBS:atmel
-LIBS:contrib
-LIBS:valves
-LIBS:relays
-LIBS:sensors
-LIBS:nxp_armmcu
 LIBS:dc-dc
-LIBS:powerint
-LIBS:Power_Management
-LIBS:ab2_connectivity
-LIBS:ab2_idc
-LIBS:ab2_terminal_block
+LIBS:sunpowered-cache
 EELAYER 25 0
 EELAYER END
 $Descr A4 11693 8268
 encoding utf-8
-Sheet 2 2
+Sheet 2 3
 Title "Sunpowered Input Board"
 Date ""
@@
 $EndComp
 $Comp
-L GNDD #PWR01
+L GNDD #PWR05
 U 1 1 55E0DA4C
 P 3450 2300
-F 0 "#PWR01" H 3450 2050 60  0001 C CNN
+F 0 "#PWR05" H 3450 2050 60  0001 C CNN
 F 1 "GNDD" H 3450 2150 60  0000 C CNN
 F 2 "" H 3450 2300 60  0000 C CNN
@@
 PowerOn
 $Comp
-L GNDD #PWR02
+L GNDD #PWR06
 U 1 1 55E0DA5C
 P 4600 2350
-F 0 "#PWR02" H 4600 2100 60  0001 C CNN
+F 0 "#PWR06" H 4600 2100 60  0001 C CNN
 F 1 "GNDD" H 4600 2200 60  0000 C CNN
 F 2 "" H 4600 2350 60  0000 C CNN
@@
 $EndComp
 $Comp
-L PWR_FLAG #FLG03
+L PWR_FLAG #FLG07
 U 1 1 55E0DA69
 P 4200 1300
-F 0 "#FLG03" H 4200 1395 30  0001 C CNN
+F 0 "#FLG07" H 4200 1395 30  0001 C CNN
 F 1 "PWR_FLAG" H 4200 1480 30  0001 C CNN
 F 2 "" H 4200 1300 60  0000 C CNN
@@
 $EndComp
 $Comp
-L +5V #PWR04
+L +5V #PWR08
 U 1 1 55E0DA6F
 P 2850 1600
-F 0 "#PWR04" H 2850 1450 60  0001 C CNN
+F 0 "#PWR08" H 2850 1450 60  0001 C CNN
 F 1 "+5V" H 2850 1740 60  0000 C CNN
 F 2 "" H 2850 1600 60  0000 C CNN
@@
 Connection ~ 6500 2650
 Wire Wire Line
-	5350 2200 5350 2650
+	5350 2650 5350 2200
 Connection ~ 5350 2650
 Wire Wire Line
@@
 	3250 1700 3600 1700
 Wire Wire Line
-	3450 2300 3450 2200
+	3450 2150 3450 2300
 Wire Wire Line
 	3450 1700 3450 1850
@@
 	2850 1600 2850 1700
 $Comp
-L PWR_FLAG #FLG05
+L PWR_FLAG #FLG09
 U 1 1 55E0DAAC
 P 2650 1300
-F 0 "#FLG05" H 2650 1395 30  0001 C CNN
+F 0 "#FLG09" H 2650 1395 30  0001 C CNN
 F 1 "PWR_FLAG" H 2650 1480 30  0001 C CNN
 F 2 "" H 2650 1300 60  0000 C CNN
@@
 15mA
 $Comp
-L PWR_FLAG #FLG06
+L PWR_FLAG #FLG010
 U 1 1 55E0DAB3
 P 3450 1700
-F 0 "#FLG06" H 3450 1795 30  0001 C CNN
+F 0 "#FLG010" H 3450 1795 30  0001 C CNN
 F 1 "PWR_FLAG" H 3450 1880 30  0001 C CNN
 F 2 "" H 3450 1700 60  0000 C CNN
@@
 Text GLabel 1550 3900 0    60   Output ~ 0
 PowerOn
-Text GLabel 2300 4650 3    60   Input ~ 0
+Text GLabel 2300 4500 3    60   Output ~ 0
 PanelVoltageSense-
 Text GLabel 2850 4650 3    60   Input ~ 0
 PanelVoltageSense+
 $Comp
-L +5V #PWR07
+L +5V #PWR011
 U 1 1 55E0DF60
-P 3350 3900
-F 0 "#PWR07" H 3350 3750 60  0001 C CNN
-F 1 "+5V" H 3350 4040 60  0000 C CNN
-F 2 "" H 3350 3900 60  0000 C CNN
-F 3 "" H 3350 3900 60  0000 C CNN
-	1    3350 3900
+P 3350 3800
+F 0 "#PWR011" H 3350 3650 60  0001 C CNN
+F 1 "+5V" H 3350 3940 60  0000 C CNN
+F 2 "" H 3350 3800 60  0000 C CNN
+F 3 "" H 3350 3800 60  0000 C CNN
+	1    3350 3800
 	1    0    0    -1
 $EndComp
 Wire Wire Line
 	2200 3900 3350 3900
-$Comp
-L PWR_FLAG #FLG08
-U 1 1 55E0DF67
-P 3050 3900
-F 0 "#FLG08" H 3050 3995 30  0001 C CNN
-F 1 "PWR_FLAG" H 3050 4080 30  0001 C CNN
-F 2 "" H 3050 3900 60  0000 C CNN
-F 3 "" H 3050 3900 60  0000 C CNN
-	1    3050 3900
-	1    0    0    -1
-$EndComp
-Connection ~ 3050 3900
 Text GLabel 2650 4650 3    60   Input ~ 0
 CurrentSensorVoltageSense
@@
 Connection ~ 1700 4000
 $Comp
-L GNDD #PWR09
+L GNDD #PWR012
 U 1 1 55E0DF80
 P 1700 4550
-F 0 "#PWR09" H 1700 4300 60  0001 C CNN
+F 0 "#PWR012" H 1700 4300 60  0001 C CNN
 F 1 "GNDD" H 1700 4400 60  0000 C CNN
 F 2 "" H 1700 4550 60  0000 C CNN
@@
 	2200 4100 2650 4100
 Wire Wire Line
-	2300 4650 2300 4300
+	2300 4500 2300 4300
 Wire Wire Line
 	2300 4300 2200 4300
@@
 Wire Wire Line
 	2500 4200 2500 4650
-Text GLabel 1350 4300 0    60   BiDi ~ 0
-DigitalGround
-Wire Wire Line
-	1350 4300 1700 4300
-Wire Wire Line
-	7950 2150 7850 2150
+Wire Wire Line
+	1700 4300 1350 4300
+Wire Wire Line
+	7850 2150 7950 2150
 Wire Wire Line
 	7450 2150 7450 2250
@@
 Wire Wire Line
 	6500 1800 6500 1300
-Text GLabel 2200 3850 1    60   BiDi ~ 0
-+5V
-Wire Wire Line
-	2200 3850 2200 3900
-Connection ~ 2200 3900
 $Comp
 L D_Schottky D2
@@
 Wire Wire Line
 	1700 4000 1700 4550
+Text HLabel 8450 1300 1    60   Output ~ 0
+RawPositive
+Text HLabel 8500 1650 2    60   Output ~ 0
+RawGround
+Text HLabel 3000 3800 1    60   BiDi ~ 0
++5V
+Text HLabel 1350 4300 0    60   BiDi ~ 0
+GNDD
+Wire Wire Line
+	3000 3800 3000 3900
+Connection ~ 3000 3900
+Wire Wire Line
+	3350 3900 3350 3800
 $EndSCHEMATC
